File: GH LP Wii.kicad_sch (KiCad schematic)
At the start: 0 parts

Commit message: uhh mostly done I guess
Parts:
- added A1: RaspberryPi_Pico, Module:RaspberryPi_Pico_Common_Unspecified, symbol MCU_Module:RaspberryPi_Pico
- added Neck1: ~, Library:Frets, symbol Symbols:neck_connection
- added RV1: R_Potentiometer, Library:Whammy Pot, symbol Device:R_Potentiometer
- added SW1: SW_Push_Dual, symbol Switch:SW_Push_Dual
- added SW_DOWN1, SW_UP1: SW_Push_45deg, PCM_Switch_Keyboard_Alps_Matias:SW_Alps_Matias, symbol Switch:SW_Push_45deg
Connections:
- new net: A1.1 (GPIO0), Neck1.1 (Green)
- new net: A1.2 (GPIO1), Neck1.2 (Red)
- new net: A1.4 (GPIO2), Neck1.3 (Yellow)
- new net: A1.11 (GPIO8), Neck1.4 (Blue)
- new net: A1.12 (GPIO9), Neck1.5 (Orange)
- new net: A1.13 (GND), A1.18 (GND), A1.23 (GND), A1.28 (GND), A1.3 (GND), A1.38 (GND), A1.8 (GND), Neck1.6 (GND), SW1.2, SW1.4, SW_DOWN1.1, SW_UP1.1
- new net: A1.14 (GPIO10), SW_DOWN1.2
- new net: A1.21 (GPIO16), SW1.1
- new net: A1.22 (GPIO17), SW1.3
- new net: A1.31 (GPIO26_ADC0), RV1.1
- new net: A1.32 (GPIO27_ADC1), RV1.2
- new net: A1.33 (AGND), RV1.3
- new net: A1.7 (GPIO5), SW_UP1.2
